File: badge.kicad_sch (KiCad schematic)
At the start: 33 parts, among them J1 SAO V.1.69bis master, Q1 BSS138, SW1 power, SW2 SW_Push, SW3 update epaper, U1 Seeed XIAO ESP32-C3, U2 MH-ET_epaper_ 2.13, U3 5V boost converter, U4 TXS0104EPWR

Commit message: reverse polarity of battery connector
Connections:
- net at SW1.1 (A): now also BT1.2 (+); no longer BT1.1 (+)
- net at SW1.4 (A): now also BT1.1 (-); no longer BT1.2 (-)
Changed lines of the file:
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@@
       (effects (font (size 1.27 1.27)) (justify left))
     )
-    (property "Footprint" "Connector_JST:JST_PH_S2B-PH-SM4-TB_1x02-1MP_P2.00mm_Horizontal" (id 2) (at 25.4 84.836 90)
+    (property "Footprint" "Connector_JST:JST_PH_S2B-PH-SM4-TB_1x02-1MP_P2.00mm_Horizontal" (id 2) (at 29.21 85.09 90)
       (effects (font (size 1.27 1.27)) hide)
     )
@@
       (effects (font (size 1.27 1.27)) hide)
     )
+    (pin "2")
     (pin "1")
-    (pin "2")
   )
   (symbol (lib_id "power:GND") (at 142.24 63.5 0) (unit 1)

Commit message: avoid shorting battery-charge output
Connections:
- net GND: no longer SW1.3 (C)
Changed lines of the file:
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@@
   (junction (at 247.65 105.41) (diameter 0) (color 0 0 0 0)
   )
-  (junction (at 30.48 100.33) (diameter 0) (color 0 0 0 0)
-  )
   (junction (at 57.15 81.28) (diameter 0) (color 0 0 0 0)
   )
@@
   )
   (wire (pts (xy 146.05 24.13) (xy 146.05 45.72))
-    (stroke (width 0) (type default) (color 0 0 0 0))
-  )
-  (wire (pts (xy 30.48 83.82) (xy 30.48 100.33))
     (stroke (width 0) (type default) (color 0 0 0 0))
   )
@@
       (effects (font (size 1.27 1.27)) hide)
     )
-    (pin "2")
-    (pin "1")
+    (pin "1")
+    (pin "2")
   )
   (symbol (lib_id "power:GND") (at 142.24 63.5 0) (unit 1)
