File: hardware/badge.kicad_sch (KiCad schematic)
At the start: 50 parts, among them J1 SAO V.1.69bis host, SW1 power, SW2 SW_Push, SW3 update epaper, U1 Seeed XIAO ESP32-C3, U2 MH-ET_epaper_ 2.13, U3 5V boost converter, U4 TXS0104EPWR

Commit message: move EPD /cs from OE to Vdark
Connections:
- net OE/cs renamed OE
- net OE: no longer U2.4 (~{CS})
- net Vdark renamed Vdark/cs
- net Vdark/cs: now also U2.4 (~{CS})
Changed lines of the file:
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@@
 		)
 	)
-	(label "OE{slash}cs"
+	(text_box "light 2k5\ndark 35k"
+		(exclude_from_sim no)
+		(at 48.26 143.51 0)
+		(size 11.43 6.35)
+		(stroke
+			(width 0)
+			(type default)
+		)
+		(fill
+			(type none)
+		)
+		(effects
+			(font
+				(size 1.27 1.27)
+			)
+			(justify left top)
+		)
+	)
+	(label "OE"
 		(at 127 60.96 0)
 		(fields_autoplaced yes)
@@
 		)
 	)
-	(label "Vdark"
+	(label "Vdark{slash}cs"
 		(at 59.69 49.53 0)
 		(fields_autoplaced yes)
@@
 		)
 	)
-	(label "OE{slash}cs"
+	(label "OE"
 		(at 147.32 111.76 0)
 		(fields_autoplaced yes)
@@
 		)
 	)
-	(label "OE{slash}cs"
+	(label "Vdark{slash}cs"
 		(at 231.14 49.53 0)
 		(fields_autoplaced yes)
@@
 		)
 	)
-	(label "Vdark"
+	(label "Vdark{slash}cs"
 		(at 48.26 135.89 0)
 		(fields_autoplaced yes)

Commit message: officially change LED current-limiter to 100R
Parts:
- R11: value 150 -> 100
Changed lines of the file:
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@@
 			)
 		)
-		(property "Value" "150"
+		(property "Value" "100"
 			(at 195.58 146.0499 0)
 			(effects
